Commit message: fixed warning issues. deleted hand_ links/joints. added gripper. added colors. fixed upper/lower limit.

File: gym-foodhunting/urdf/hsrb4s.urdf (robot description, URDF)
Before this commit: robot hsrb, 45 links, 44 joints
Links:
- removed link hand_camera_frame
- removed link hand_camera_gazebo_frame
- removed link hand_l_distal_link
- removed link hand_l_finger_tip_frame
- removed link hand_l_finger_vacuum_frame
- removed link hand_l_mimic_distal_link
- removed link hand_l_proximal_link
- removed link hand_l_spring_proximal_link
- removed link hand_motor_dummy_link
- removed link hand_palm_link
- removed link hand_r_distal_link
- removed link hand_r_finger_tip_frame
- removed link hand_r_mimic_distal_link
- removed link hand_r_proximal_link
- removed link hand_r_spring_proximal_link
- added link gripper_pole, mass 0.05; collision cylinder length=0.2 radius=.01; visual cylinder length=0.2 radius=.01
- added link left_gripper, mass 0.05; collision mesh filename=l_finger.stl; visual mesh filename=l_finger.stl
- added link left_tip, mass 0.05; collision mesh filename=l_finger_tip.stl; visual mesh filename=l_finger_tip.stl
- added link right_gripper, mass 0.05; collision mesh filename=l_finger.stl; visual mesh filename=l_finger.stl
- added link right_tip, mass 0.05; collision mesh filename=l_finger_tip.stl; visual mesh filename=l_finger_tip.stl
- link base_footprint: mass None -> 0.01
- link base_imu_frame: mass None -> 0.0
- link base_range_sensor_link: mass None -> 0.0
- link head_center_camera_frame: mass None -> 0.0
- link head_center_camera_gazebo_frame: mass None -> 0.0
- link head_l_stereo_camera_gazebo_frame: mass None -> 0.0
- link head_l_stereo_camera_link: mass None -> 0.0
- link head_r_stereo_camera_gazebo_frame: mass None -> 0.0
- link head_r_stereo_camera_link: mass None -> 0.0
- link head_rgbd_sensor_gazebo_frame: mass None -> 0.0
- link head_rgbd_sensor_link: mass None -> 0.0
- link wrist_ft_sensor_frame: mass None -> 0.0
Joints:
- removed joint hand_camera_frame_joint
- removed joint hand_camera_gazebo_frame_joint
- removed joint hand_l_distal_joint
- removed joint hand_l_finger_tip_frame_joint
- removed joint hand_l_finger_vacuum_frame_joint
- removed joint hand_l_mimic_distal_joint
- removed joint hand_l_proximal_joint
- removed joint hand_l_spring_proximal_joint
- removed joint hand_motor_joint
- removed joint hand_palm_joint
- removed joint hand_r_distal_joint
- removed joint hand_r_finger_tip_frame_joint
- removed joint hand_r_mimic_distal_joint
- removed joint hand_r_proximal_joint
- removed joint hand_r_spring_proximal_joint
- added joint gripper_extension: type fixed, parent wrist_roll_link, child gripper_pole, origin xyz=0 0 -0.05 rpy=0 -1.57075 0, axis 1 0 0
- added joint left_gripper_joint: type revolute, parent gripper_pole, child left_gripper, origin xyz=0.2 0.02 0 rpy=0 0 0, axis 0 0 1, limit lower=0.0 upper=0.548 effort=1000.0 velocity=0.5
- added joint left_tip_joint: type fixed, parent left_gripper, child left_tip
- added joint right_gripper_joint: type revolute, parent gripper_pole, child right_gripper, origin xyz=0.2 -0.02 0 rpy=0 0 0, axis 0 0 -1, limit lower=0.0 upper=0.548 effort=1000.0 velocity=0.5
- added joint right_tip_joint: type fixed, parent right_gripper, child right_tip
- joint arm_lift_joint: limit lower=0.0 upper=0.69 effort=100.0 velocity=0.2 -> lower=0.0 upper=0.3 effort=100.0 velocity=0.2
- joint arm_roll_joint: limit lower=-2.09 upper=3.84 effort=100.0 velocity=2.0 -> lower=-3.14159265359 upper=3.14159265359 effort=100.0 velocity=2.0
- joint base_roll_joint: limit effort=34.46 velocity=2.5 -> lower=-3.14159265359 upper=3.14159265359 effort=34.46 velocity=2.5
- joint head_pan_joint: limit lower=-3.84 upper=1.75 effort=100.0 velocity=1.0 -> lower=-3.14159265359 upper=3.14159265359 effort=100.0 velocity=1.0
- joint head_tilt_joint: limit lower=-1.57 upper=0.52 effort=100.0 velocity=1.0 -> lower=-0.78539816339 upper=0.78539816339 effort=100.0 velocity=1.0
- joint wrist_flex_joint: limit lower=-1.92 upper=1.22 effort=100.0 velocity=1.5 -> lower=-1.5707963268 upper=1.5707963268 effort=100.0 velocity=1.5
- joint wrist_roll_joint: limit lower=-1.92 upper=3.67 effort=100.0 velocity=1.5 -> lower=-3.14159265359 upper=3.14159265359 effort=100.0 velocity=1.5
